File: PCB/typring-kicad/typring-kicad.kicad_pcb (KiCad board)
At the start: 2 copper layers, 90 parts, among them J1 Conn_01x03_Female, J2 Conn_01x05_Female, J3 Conn_01x01_Female, J4 Conn_01x04_Female, J5 Conn_01x01_Female, J6 Conn_01x06_Female, J7 Conn_01x03_Female, U1 CAP_SENSE_4mm_rx-tx-_half, U10 CAP_SENSE_4mm_rx-tx-_half, U11 CAP_SENSE_4mm_rx-tx-_half, U12 CAP_SENSE_4mm_rx-tx-_whole, U13 CAP_SENSE_4mm_rx-tx-_half, U14 CAP_SENSE_4mm_rx-tx-_whole, U15 CAP_SENSE_4mm_rx-tx-_whole, U16 CAP_SENSE_4mm_rx-tx-_whole, U17 CAP_SENSE_4mm_rx-tx-_half, U18 CAP_SENSE_4mm_rx-tx-_whole, U19 CAP_SENSE_4mm_rx-tx-_whole, U2 CAP_SENSE_4mm_rx-tx-_whole, U20 CAP_SENSE_4mm_rx-tx-_whole, U21 CAP_SENSE_4mm_rx-tx-_whole, U22 CAP_SENSE_4mm_rx-tx-_whole, U23 CAP_SENSE_4mm_rx-tx-_half, U24 CAP_SENSE_4mm_rx-tx-_whole, U25 CAP_SENSE_4mm_rx-tx-_half, U26 CAP_SENSE_4mm_rx-tx-_whole, U27 CAP_SENSE_4mm_rx-tx-_half, U28 CAP_SENSE_4mm_rx-tx-_whole, U29 CAP_SENSE_4mm_rx-tx-_half, U3 CAP_SENSE_4mm_rx-tx-_whole, U30 CAP_SENSE_4mm_rx-tx-_whole, U31 CAP_SENSE_4mm_rx-tx-_half, U32 CAP_SENSE_4mm_rx-tx-_half, U33 CAP_SENSE_4mm_rx-tx-_half, U34 CAP_SENSE_4mm_rx-tx-_whole, U35 CAP_SENSE_4mm_rx-tx-_whole, U36 CAP_SENSE_4mm_rx-tx-_whole, U37 CAP_SENSE_4mm_rx-tx-_whole, U38 CAP_SENSE_4mm_rx-tx-_whole, U4 CAP_SENSE_4mm_rx-tx-_whole, U48 CAP_SENSE_3.5mm_rx-tx-_half, U49 CAP_SENSE_3.5mm_rx-tx-_half, U5 CAP_SENSE_4mm_rx-tx-_whole, U50 CAP_SENSE_3.5mm_rx-tx-_half, U51 CAP_SENSE_3.5mm_rx-tx-_half, U52 CAP_SENSE_3.5mm_rx-tx-_half, U53 CAP_SENSE_3.5mm_rx-tx-_half, U54 CAP_SENSE_3.5mm_rx-tx-_whole, U56 CAP_SENSE_3.5mm_rx-tx-_half, U58 CAP_SENSE_3.5mm_rx-tx-_whole, U6 CAP_SENSE_4mm_rx-tx-_half, U60 CAP_SENSE_3.5mm_rx-tx-_whole, U62 CAP_SENSE_3.5mm_rx-tx-_whole, U63 CAP_SENSE_3.5mm_rx-tx-_whole, U64 CAP_SENSE_3.5mm_rx-tx-_whole, U65 CAP_SENSE_3.5mm_rx-tx-_whole, U66 CAP_SENSE_3.5mm_rx-tx-_half, U67 CAP_SENSE_3.5mm_rx-tx-_whole, U68 CAP_SENSE_3.5mm_rx-tx-_whole, U69 CAP_SENSE_3.5mm_rx-tx-_half, U7 CAP_SENSE_4mm_rx-tx-_half, U70 CAP_SENSE_3.5mm_rx-tx-_whole, U71 CAP_SENSE_3.5mm_rx-tx-_whole, U72 CAP_SENSE_3.5mm_rx-tx-_whole, U73 CAP_SENSE_3.5mm_rx-tx-_whole, U74 CAP_SENSE_3.5mm_rx-tx-_whole, U75 CAP_SENSE_3.5mm_rx-tx-_whole, U76 CAP_SENSE_3.5mm_rx-tx-_whole, U77 CAP_SENSE_3.5mm_rx-tx-_whole, U78 CAP_SENSE_3.5mm_rx-tx-_half, U79 CAP_SENSE_3.5mm_rx-tx-_whole, U8 CAP_SENSE_4mm_rx-tx-_half, U80 CAP_SENSE_3.5mm_rx-tx-_whole, U81 CAP_SENSE_3.5mm_rx-tx-_half, U82 CAP_SENSE_3.5mm_rx-tx-_whole, U83 CAP_SENSE_3.5mm_rx-tx-_whole, U84 CAP_SENSE_3.5mm_rx-tx-_whole, U85 CAP_SENSE_3.5mm_rx-tx-_whole, U86 CAP_SENSE_3.5mm_rx-tx-_half, U87 CAP_SENSE_3.5mm_rx-tx-_half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

Commit message: add final size, gerbers, drill file
Parts:
- added J8: Conn_01x01_Female, Connector_PinHeader_2.54mm:PinHeader_1x01_P2.54mm_Vertical, F.Cu at (145.0, 22.2)
- added J9: Conn_01x07_Female, Connector_PinHeader_2.54mm:PinHeader_1x07_P2.54mm_Vertical, F.Cu at (145.3, 33.0)
- added U100: CAP_SENSE_3mm_rx-tx-_whole, cap_sense:CAP_SENSE_3.0mm_rx-tx_whole, F.Cu at (170.8, 44.8)
- added U101: CAP_SENSE_3mm_rx-tx-_half, cap_sense:CAP_SENSE_3.0mm_rx-tx_half, F.Cu at (172.5, 49.8)
- added U102: CAP_SENSE_3mm_rx-tx-_whole, cap_sense:CAP_SENSE_3.0mm_rx-tx_whole, F.Cu at (174.1, 41.5)
- added U103: CAP_SENSE_3mm_rx-tx-_whole, cap_sense:CAP_SENSE_3.0mm_rx-tx_whole, F.Cu at (167.5, 48.1)
- added U104: CAP_SENSE_3mm_rx-tx-_whole, cap_sense:CAP_SENSE_3.0mm_rx-tx_whole, F.Cu at (167.5, 28.1)
- added U105: CAP_SENSE_3mm_rx-tx-_half, cap_sense:CAP_SENSE_3.0mm_rx-tx_half, F.Cu at (165.6, 49.6)
- added U106: CAP_SENSE_3mm_rx-tx-_whole, cap_sense:CAP_SENSE_3.0mm_rx-tx_whole, F.Cu at (175.8, 46.5)
- added U107: CAP_SENSE_3mm_rx-tx-_whole, cap_sense:CAP_SENSE_3.0mm_rx-tx_whole, F.Cu at (174.1, 48.1)
- added U108: CAP_SENSE_3mm_rx-tx-_whole, cap_sense:CAP_SENSE_3.0mm_rx-tx_whole, F.Cu at (170.8, 48.1)
- added U109: CAP_SENSE_3mm_rx-tx-_whole, cap_sense:CAP_SENSE_3.0mm_rx-tx_whole, F.Cu at (169.1, 43.1)
- added U110: CAP_SENSE_3mm_rx-tx-_whole, cap_sense:CAP_SENSE_3.0mm_rx-tx_whole, F.Cu at (167.5, 44.8)
- added U111: CAP_SENSE_3mm_rx-tx-_whole, cap_sense:CAP_SENSE_3.0mm_rx-tx_whole, F.Cu at (174.1, 44.8)
- added U112: CAP_SENSE_3mm_rx-tx-_whole, cap_sense:CAP_SENSE_3.0mm_rx-tx_whole, F.Cu at (175.8, 39.8)
- added U113: CAP_SENSE_3mm_rx-tx-_half, cap_sense:CAP_SENSE_3.0mm_rx-tx_half, F.Cu at (175.8, 29.4)
- added U114: CAP_SENSE_3mm_rx-tx-_whole, cap_sense:CAP_SENSE_3.0mm_rx-tx_whole, F.Cu at (165.8, 33.1)
- added U115: CAP_SENSE_3mm_rx-tx-_whole, cap_sense:CAP_SENSE_3.0mm_rx-tx_whole, F.Cu at (165.8, 43.1)
- added U116: CAP_SENSE_3mm_rx-tx-_whole, cap_sense:CAP_SENSE_3.0mm_rx-tx_whole, F.Cu at (172.5, 33.1)
- added U117: CAP_SENSE_3mm_rx-tx-_whole, cap_sense:CAP_SENSE_3.0mm_rx-tx_whole, F.Cu at (174.1, 34.8)
- added U118: CAP_SENSE_3mm_rx-tx-_whole, cap_sense:CAP_SENSE_3.0mm_rx-tx_whole, F.Cu at (174.1, 38.1)
- added U119: CAP_SENSE_3mm_rx-tx-_whole, cap_sense:CAP_SENSE_3.0mm_rx-tx_whole, F.Cu at (172.5, 43.1)
- added U120: CAP_SENSE_3mm_rx-tx-_half, cap_sense:CAP_SENSE_3.0mm_rx-tx_half, F.Cu at (165.8, 29.4)
- added U121: CAP_SENSE_3mm_rx-tx-_whole, cap_sense:CAP_SENSE_3.0mm_rx-tx_whole, F.Cu at (165.8, 36.5)
- added U122: CAP_SENSE_3mm_rx-tx-_half, cap_sense:CAP_SENSE_3.0mm_rx-tx_half, F.Cu at (169.1, 49.8)
- added U123: CAP_SENSE_3mm_rx-tx-_whole, cap_sense:CAP_SENSE_3.0mm_rx-tx_whole, F.Cu at (172.5, 46.5)
- added U124: CAP_SENSE_3mm_rx-tx-_whole, cap_sense:CAP_SENSE_3.0mm_rx-tx_whole, F.Cu at (169.1, 36.5)
- added U125: CAP_SENSE_3mm_rx-tx-_whole, cap_sense:CAP_SENSE_3.0mm_rx-tx_whole, F.Cu at (169.1, 33.1)
- added U126: CAP_SENSE_3mm_rx-tx-_whole, cap_sense:CAP_SENSE_3.0mm_rx-tx_whole, F.Cu at (167.5, 31.5)
- added U127: CAP_SENSE_3mm_rx-tx-_whole, cap_sense:CAP_SENSE_3.0mm_rx-tx_whole, F.Cu at (165.8, 39.8)
- added U128: CAP_SENSE_3mm_rx-tx-_whole, cap_sense:CAP_SENSE_3.0mm_rx-tx_whole, F.Cu at (175.8, 29.8)
- added U129: CAP_SENSE_3mm_rx-tx-_whole, cap_sense:CAP_SENSE_3.0mm_rx-tx_whole, F.Cu at (170.8, 31.5)
- added U130: CAP_SENSE_3mm_rx-tx-_whole, cap_sense:CAP_SENSE_3.0mm_rx-tx_whole, F.Cu at (175.8, 36.5)
- added U131: CAP_SENSE_3mm_rx-tx-_whole, cap_sense:CAP_SENSE_3.0mm_rx-tx_whole, F.Cu at (167.5, 38.1)
- added U132: CAP_SENSE_3mm_rx-tx-_whole, cap_sense:CAP_SENSE_3.0mm_rx-tx_whole, F.Cu at (167.5, 34.8)
- added U133: CAP_SENSE_3mm_rx-tx-_whole, cap_sense:CAP_SENSE_3.0mm_rx-tx_whole, F.Cu at (165.8, 29.8)
- added U134: CAP_SENSE_3mm_rx-tx-_whole, cap_sense:CAP_SENSE_3.0mm_rx-tx_whole, F.Cu at (172.5, 36.5)
- added U135: CAP_SENSE_3mm_rx-tx-_half, cap_sense:CAP_SENSE_3.0mm_rx-tx_half, F.Cu at (176.0, 32.9)
- added U136: CAP_SENSE_3mm_rx-tx-_half, cap_sense:CAP_SENSE_3.0mm_rx-tx_half, F.Cu at (165.6, 36.3)
- added U137: CAP_SENSE_3mm_rx-tx-_whole, cap_sense:CAP_SENSE_3.0mm_rx-tx_whole, F.Cu at (174.1, 31.5)
- added U138: CAP_SENSE_3mm_rx-tx-_whole, cap_sense:CAP_SENSE_3.0mm_rx-tx_whole, F.Cu at (175.6, 29.6)
- added U139: CAP_SENSE_3mm_rx-tx-_whole, cap_sense:CAP_SENSE_3.0mm_rx-tx_whole, F.Cu at (169.1, 29.8)
- added U140: CAP_SENSE_3mm_rx-tx-_whole, cap_sense:CAP_SENSE_3.0mm_rx-tx_whole, F.Cu at (175.8, 33.1)
- added U141: CAP_SENSE_3mm_rx-tx-_whole, cap_sense:CAP_SENSE_3.0mm_rx-tx_whole, F.Cu at (172.5, 29.8)
- added U142: CAP_SENSE_3mm_rx-tx-_whole, cap_sense:CAP_SENSE_3.0mm_rx-tx_whole, F.Cu at (170.8, 34.8)
- added U143: CAP_SENSE_3mm_rx-tx-_half, cap_sense:CAP_SENSE_3.0mm_rx-tx_half, F.Cu at (176.0, 39.6)
- added U144: CAP_SENSE_3mm_rx-tx-_half, cap_sense:CAP_SENSE_3.0mm_rx-tx_half, F.Cu at (175.8, 49.8)
- added U145: CAP_SENSE_3mm_rx-tx-_half, cap_sense:CAP_SENSE_3.0mm_rx-tx_half, F.Cu at (176.0, 36.3)
- added U146: CAP_SENSE_3mm_rx-tx-_half, cap_sense:CAP_SENSE_3.0mm_rx-tx_half, F.Cu at (165.6, 39.6)
- added U147: CAP_SENSE_3mm_rx-tx-_half, cap_sense:CAP_SENSE_3.0mm_rx-tx_half, F.Cu at (176.0, 29.6)
- added U148: CAP_SENSE_3mm_rx-tx-_half, cap_sense:CAP_SENSE_3.0mm_rx-tx_half, F.Cu at (176.0, 42.9)
- added U149: CAP_SENSE_3mm_rx-tx-_half, cap_sense:CAP_SENSE_3.0mm_rx-tx_half, F.Cu at (165.6, 46.3)
- added U150: CAP_SENSE_3mm_rx-tx-_half, cap_sense:CAP_SENSE_3.0mm_rx-tx_half, F.Cu at (172.5, 29.4)
- added U39: CAP_SENSE_3mm_rx-tx-_whole, cap_sense:CAP_SENSE_3.0mm_rx-tx_whole, F.Cu at (175.8, 43.1)
- added U40: CAP_SENSE_3mm_rx-tx-_half, cap_sense:CAP_SENSE_3.0mm_rx-tx_half, F.Cu at (169.1, 29.4)
- added U41: CAP_SENSE_3mm_rx-tx-_whole, cap_sense:CAP_SENSE_3.0mm_rx-tx_whole, F.Cu at (172.3, 29.6)
- added U42: CAP_SENSE_3mm_rx-tx-_whole, cap_sense:CAP_SENSE_3.0mm_rx-tx_whole, F.Cu at (169.1, 39.8)
- added U43: CAP_SENSE_3mm_rx-tx-_whole, cap_sense:CAP_SENSE_3.0mm_rx-tx_whole, F.Cu at (167.5, 41.5)
- added U44: CAP_SENSE_3mm_rx-tx-_half, cap_sense:CAP_SENSE_3.0mm_rx-tx_half, F.Cu at (176.0, 46.3)
- added U45: CAP_SENSE_3mm_rx-tx-_whole, cap_sense:CAP_SENSE_3.0mm_rx-tx_whole, F.Cu at (165.8, 46.5)
- added U46: CAP_SENSE_3mm_rx-tx-_half, cap_sense:CAP_SENSE_3.0mm_rx-tx_half, F.Cu at (165.6, 29.6)
- added U47: CAP_SENSE_3mm_rx-tx-_whole, cap_sense:CAP_SENSE_3.0mm_rx-tx_whole, F.Cu at (170.8, 41.5)
- added U55: CAP_SENSE_3mm_rx-tx-_half, cap_sense:CAP_SENSE_3.0mm_rx-tx_half, F.Cu at (165.8, 49.8)
- added U57: CAP_SENSE_3mm_rx-tx-_whole, cap_sense:CAP_SENSE_3.0mm_rx-tx_whole, F.Cu at (170.8, 38.1)
- added U59: CAP_SENSE_3mm_rx-tx-_half, cap_sense:CAP_SENSE_3.0mm_rx-tx_half, F.Cu at (165.6, 42.9)
- added U61: CAP_SENSE_3mm_rx-tx-_half, cap_sense:CAP_SENSE_3.0mm_rx-tx_half, F.Cu at (165.6, 32.9)
- added U97: CAP_SENSE_3mm_rx-tx-_whole, cap_sense:CAP_SENSE_3.0mm_rx-tx_whole, F.Cu at (169.1, 46.5)
- added U98: CAP_SENSE_3mm_rx-tx-_whole, cap_sense:CAP_SENSE_3.0mm_rx-tx_whole, F.Cu at (172.5, 39.8)
- added U99: CAP_SENSE_3mm_rx-tx-_half, cap_sense:CAP_SENSE_3.0mm_rx-tx_half, F.Cu at (176.0, 49.6)
- moved J4 13.1 mm to (154.1, 22.0)
Routing:
- net GND: track 114.0 -> 385.5 mm, vias 19 -> 61
- net (no net): track 24.0 -> 118.2 mm, vias 30 -> 122
- net Net-(J6-Pad1): track 0.00 -> 22.6 mm
- net Net-(J6-Pad2): track 0.00 -> 22.2 mm
- net Net-(J6-Pad3): track 0.00 -> 21.6 mm
- net Net-(J6-Pad6): track 0.00 -> 21.0 mm
- net Net-(J6-Pad4): track 0.00 -> 20.9 mm
- net Net-(J9-Pad1): track 0.00 -> 20.5 mm
- net Net-(J6-Pad5): track 0.00 -> 20.4 mm
- net Net-(J9-Pad2): track 0.00 -> 20.1 mm
- net Net-(J9-Pad3): track 0.00 -> 19.9 mm
- net Net-(J9-Pad7): track 0.00 -> 19.6 mm
- net Net-(J9-Pad4): track 0.00 -> 19.5 mm
- net Net-(J9-Pad5): track 0.00 -> 19.1 mm
- net Net-(J9-Pad6): track 0.00 -> 19.1 mm
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- removed copper zone on B.Cu, net (none)
Other:
- board outline added: 112.5 x 35.5 mm
