File: PCB/typring-kicad/typring-kicad.sch (KiCad schematic (older format))
At the start: 90 parts, among them J1 Conn_01x03_Female, J2 Conn_01x05_Female, J3 Conn_01x01_Female, J4 Conn_01x04_Female, J5 Conn_01x01_Female, J6 Conn_01x06_Female, J7 Conn_01x03_Female, U1 CAP_SENSE_4mm_rx-tx-_half, U10 CAP_SENSE_4mm_rx-tx-_half, U11 CAP_SENSE_4mm_rx-tx-_half, U12 CAP_SENSE_4mm_rx-tx-_whole, U13 CAP_SENSE_4mm_rx-tx-_half, U14 CAP_SENSE_4mm_rx-tx-_whole, U15 CAP_SENSE_4mm_rx-tx-_whole, U16 CAP_SENSE_4mm_rx-tx-_whole, U17 CAP_SENSE_4mm_rx-tx-_half, U18 CAP_SENSE_4mm_rx-tx-_whole, U19 CAP_SENSE_4mm_rx-tx-_whole, U2 CAP_SENSE_4mm_rx-tx-_whole, U20 CAP_SENSE_4mm_rx-tx-_whole, U21 CAP_SENSE_4mm_rx-tx-_whole, U22 CAP_SENSE_4mm_rx-tx-_whole, U23 CAP_SENSE_4mm_rx-tx-_half, U24 CAP_SENSE_4mm_rx-tx-_whole, U25 CAP_SENSE_4mm_rx-tx-_half, U26 CAP_SENSE_4mm_rx-tx-_whole, U27 CAP_SENSE_4mm_rx-tx-_half, U28 CAP_SENSE_4mm_rx-tx-_whole, U29 CAP_SENSE_4mm_rx-tx-_half, U3 CAP_SENSE_4mm_rx-tx-_whole, U30 CAP_SENSE_4mm_rx-tx-_whole, U31 CAP_SENSE_4mm_rx-tx-_half, U32 CAP_SENSE_4mm_rx-tx-_half, U33 CAP_SENSE_4mm_rx-tx-_half, U34 CAP_SENSE_4mm_rx-tx-_whole, U35 CAP_SENSE_4mm_rx-tx-_whole, U36 CAP_SENSE_4mm_rx-tx-_whole, U37 CAP_SENSE_4mm_rx-tx-_whole, U38 CAP_SENSE_4mm_rx-tx-_whole, U4 CAP_SENSE_4mm_rx-tx-_whole, U48 CAP_SENSE_3.5mm_rx-tx-_half, U49 CAP_SENSE_3.5mm_rx-tx-_half, U5 CAP_SENSE_4mm_rx-tx-_whole, U50 CAP_SENSE_3.5mm_rx-tx-_half, U51 CAP_SENSE_3.5mm_rx-tx-_half, U52 CAP_SENSE_3.5mm_rx-tx-_half, U53 CAP_SENSE_3.5mm_rx-tx-_half, U54 CAP_SENSE_3.5mm_rx-tx-_whole, U56 CAP_SENSE_3.5mm_rx-tx-_half, U58 CAP_SENSE_3.5mm_rx-tx-_whole, U6 CAP_SENSE_4mm_rx-tx-_half, U60 CAP_SENSE_3.5mm_rx-tx-_whole, U62 CAP_SENSE_3.5mm_rx-tx-_whole, U63 CAP_SENSE_3.5mm_rx-tx-_whole, U64 CAP_SENSE_3.5mm_rx-tx-_whole, U65 CAP_SENSE_3.5mm_rx-tx-_whole, U66 CAP_SENSE_3.5mm_rx-tx-_half, U67 CAP_SENSE_3.5mm_rx-tx-_whole, U68 CAP_SENSE_3.5mm_rx-tx-_whole, U69 CAP_SENSE_3.5mm_rx-tx-_half, U7 CAP_SENSE_4mm_rx-tx-_half, U70 CAP_SENSE_3.5mm_rx-tx-_whole, U71 CAP_SENSE_3.5mm_rx-tx-_whole, U72 CAP_SENSE_3.5mm_rx-tx-_whole, U73 CAP_SENSE_3.5mm_rx-tx-_whole, U74 CAP_SENSE_3.5mm_rx-tx-_whole, U75 CAP_SENSE_3.5mm_rx-tx-_whole, U76 CAP_SENSE_3.5mm_rx-tx-_whole, U77 CAP_SENSE_3.5mm_rx-tx-_whole, U78 CAP_SENSE_3.5mm_rx-tx-_half, U79 CAP_SENSE_3.5mm_rx-tx-_whole, U8 CAP_SENSE_4mm_rx-tx-_half, U80 CAP_SENSE_3.5mm_rx-tx-_whole, U81 CAP_SENSE_3.5mm_rx-tx-_half, U82 CAP_SENSE_3.5mm_rx-tx-_whole, U83 CAP_SENSE_3.5mm_rx-tx-_whole, U84 CAP_SENSE_3.5mm_rx-tx-_whole, U85 CAP_SENSE_3.5mm_rx-tx-_whole, U86 CAP_SENSE_3.5mm_rx-tx-_half, U87 CAP_SENSE_3.5mm_rx-tx-_half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

Commit message: add final size, gerbers, drill file
Parts:
- added J8: Conn_01x01_Female, Connector_PinHeader_2.54mm:PinHeader_1x01_P2.54mm_Vertical, symbol Connector:Conn_01x01_Female
- added J9: Conn_01x07_Female, Connector_PinHeader_2.54mm:PinHeader_1x07_P2.54mm_Vertical, symbol Connector:Conn_01x07_Female
- added U100, U102, U103, U104, U106, U107, U108, U109, U110, U111, U112, U114, U115, U116, U117, U118, U119, U121, U123, U124, U125, U126, U127, U128, U129, U130, U131, U132, U133, U134, U137, U138, U139, U140, U141, U142, U39, U41, U42, U43, U45, U47, U57, U97, U98: CAP_SENSE_3mm_rx-tx-_whole, cap_sense:CAP_SENSE_3.0mm_rx-tx_whole, symbol cap_sense:CAP_SENSE_3mm_rx-tx-_whole
- added U101, U105, U113, U120, U122, U135, U136, U143, U144, U145, U146, U147, U148, U149, U150, U40, U44, U46, U55, U59, U61, U99: CAP_SENSE_3mm_rx-tx-_half, cap_sense:CAP_SENSE_3.0mm_rx-tx_half, symbol cap_sense:CAP_SENSE_3mm_rx-tx-_half
Other:
- moved on the sheet: J4, J5, J6
